File: WroomMINI.kicad_pcb (KiCad board)
At the start: 2 copper layers, 24.1 x 43.2 mm, 9 parts, among them P1 ProgHeader, SW1 RST, SW2 BOOT, U1 ESP32-WROOM

Commit message: Add files via upload
Parts:
- added C5: 10uF, Capacitors_SMD:C_1206_HandSoldering, B.Cu at (112.0, 84.8)
- added C6: 10uF, Capacitors_SMD:C_1206_HandSoldering, B.Cu at (117.9, 76.7)
- added D1: PowerOn, LEDs:LED_1206_HandSoldering, B.Cu at (112.0, 87.6)
- added G***: LOGO, 18650:SOALogo2, B.Cu at (112.2, 93.5)
- added Pwr1: Pwr, Socket_Strips:Socket_Strip_Straight_1x02_Pitch2.54mm, F.Cu at (101.9, 85.9)
- added Pwr2: 5Vin, Socket_Strips:Socket_Strip_Straight_1x02_Pitch2.54mm, F.Cu at (122.7, 87.9)
- added R2: 10k, Resistors_SMD:R_1206_HandSoldering, B.Cu at (112.0, 82.3)
- added U2: AP111733, TO_SOT_Packages_SMD:SOT-223, B.Cu at (112.4, 76.0)
Routing:
- net +3V3: track 31.8 -> 63.2 mm
- net +5V: track 0.00 -> 23.8 mm, vias 0 -> 1
- net Net-(D1-Pad2): track 0.00 -> 8.40 mm
- net Net-(P1-Pad3): track 37.4 -> 36.8 mm
- net Net-(C4-Pad1): track 22.6 -> 23.2 mm
Other:
- board text added: "3.3v"
- board text added: "5Vin"
- board text added: "Dr CADIC Philippe @pwavrobot"
- board text added: "ESP32 Minimal Board"
