File: WroomMINI.sch (KiCad schematic (older format))
At the start: 9 parts, among them P1 ProgHeader, SW1 RST, SW2 BOOT, U1 ESP32-WROOM

Commit message: Add files via upload
Parts:
- added C5, C6: 10uF, Capacitors_SMD:C_1206_HandSoldering, symbol C_Small
- added D1: PowerOn, LEDs:LED_1206_HandSoldering, symbol Led_Small
- added Pwr1: Pwr, Socket_Strips:Socket_Strip_Straight_1x02_Pitch2.54mm, symbol CONN_01X02
- added Pwr2: 5Vin, Socket_Strips:Socket_Strip_Straight_1x02_Pitch2.54mm, symbol CONN_01X02
- added R2: 10k, Resistors_SMD:R_1206_HandSoldering, symbol R_Small
- added U2: AP111733, TO_SOT_Packages_SMD:SOT-223, symbol AP111733
Connections:
- net +3V3: now also C6.1, Pwr1.1 (P1), U2.2 (VO), U2.4 (VO)
- net GND: now also C5.2, C6.2, D1.1 (K), Pwr1.2 (P2), Pwr2.1 (P1), U2.1 (GND/ADJ)
- new net: D1.2 (A), R2.2
- new net +5V: C5.1, Pwr2.2 (P2), R2.1, U2.3 (VI)
